File: PX4FMUv2.4.6.kicad_pcb (KiCad board)
At the start: 6 copper layers, 70 x 40.5 mm, 290 parts, among them J201 DF13C-6P-1.25V, J202 DF13C-6P-1.25V, J203 DF13C-6P-1.25V, J204 DF13C-6P-1.25V, J301 47346-0001, J302 DF13C-4P-1.25V, J401 DF13C-4P-1.25V, J402 DF13C-3P-1.25V, J403 DF13C-7P-1.25V, J404 DF13C-5P-1.25V, J405 DF13C-4P-1.25V, J601 DF13C-6P-1.25V, J701 DF13C-2P-1.25V, J702 DF13C-3P-1.25V, J801 JST-ZH-3, J901 HEADER-3X163X16RA, M3_MOUNT1101 MOUNT-HOLE3.1MM, M3_MOUNT1102 MOUNT-HOLE3.1MM, M3_MOUNT1103 MOUNT-HOLE3.1MM, M3_MOUNT1104 MOUNT-HOLE3.1MM, U1001 BQ24313, U1002 MIC5332, U101 STM32F4X7VX, U102 FM25V01, U1101 LTC4417, U1102 NTHD4102PT1G, U1103 NTHD4102PT1G, U1104 NTHD4102PT1G, U201 TXS0108QFN20, U202 TXS0108QFN20, U301 2908-05WB-MG, U302 NUF2042XV6, U401 MAX3051, U501 L3GD20, U502 L3GD20H, U504 LSM303D, U505 MPU-6000, U506 MS5611-01BA, U601 BQ24315, U602 BQ24315, U603 MIC5332, U701 TCA62724FMG, U702 LT3469, U703 LRTB GFTG-T7AW-1+V7A7-29+R5T9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, U801 STM32F10XCXT6, U901 TXS0108QFN20, U902 TXS0108QFN20, U903 74LVC2G240, X101 3.2x2.5 mm / 24 MHz / 15 ppm, X503 0512811094, X801 3.2x2.5 mm / 24 MHz / 15 ppm

Commit message: removed more things
Parts:
- removed C201, C401, C402, C502, C503, C507, C901, C902: 0u1, PX4FMUv2.4.6:0402-CAP
- removed C501, C506, C509, C511: 10u/10V, PX4FMUv2.4.6:0805-CAP
- removed C504, C505: 10n, PX4FMUv2.4.6:0402-CAP
- removed C510, C704: 0u47, PX4FMUv2.4.6:0402-CAP
- removed C702: 1u, PX4FMUv2.4.6:0603-CAP
- removed C703: 5n6, PX4FMUv2.4.6:0402-CAP
- removed D201, D202, D401, D402, D403, D404, D701, D901, D902: PESD0402-140, PX4FMUv2.4.6:0402-TVS
- removed J201, J202, J204: DF13C-6P-1.25V, PX4FMUv2.4.6:DF13C-6P-1.25V
- removed J302, J401, J405: DF13C-4P-1.25V, PX4FMUv2.4.6:DF13C-4P-1.25V
- removed J402, J702: DF13C-3P-1.25V, PX4FMUv2.4.6:DF13C-3P-1.25V
- removed J403: DF13C-7P-1.25V, PX4FMUv2.4.6:DF13C-7P-1.25V
- removed J404: DF13C-5P-1.25V, PX4FMUv2.4.6:DF13C-5P-1.25V
- removed J701: DF13C-2P-1.25V, PX4FMUv2.4.6:DF13C-2P-1.25V
- removed JX301, JX802: ARM_MINI_JTAG-SMT, PX4FMUv2.4.6:FTSH-105-01-XXX-DV-K
- removed JX801: HEADER-3X1BOARDEDGE-SHORT, PX4FMUv2.4.6:HEADER_3X01_SMD_H_BOARD_EDGE_SHORT
- removed L201, L202, L401, L402, L403, L404: KNH16C104DA5TS, PX4FMUv2.4.6:KYOCERA-KNH16-DA
- removed L701: 47uH, PX4FMUv2.4.6:0805-IND
- removed R201, R202, R203, R204, R208, R209, R210, R211, R404, R405, R409: 120R, PX4FMUv2.4.6:0402-RES
- removed R301, R302, R303, R304, R305, R703: 100K, PX4FMUv2.4.6:0402-RES
- removed R401, R402, R713: 1K5, PX4FMUv2.4.6:0402-RES
- removed R403, R406, R407, R408: 10K/0.1%, PX4FMUv2.4.6:0402-RES
- removed R701: 9K09, PX4FMUv2.4.6:0402-RES
- removed R702, R901: 10K, PX4FMUv2.4.6:0402-RES
- removed R705: 453K, PX4FMUv2.4.6:0402-RES
- removed R706: 16K5, PX4FMUv2.4.6:0402-RES
- removed R710: 68R, PX4FMUv2.4.6:0402-RES
- removed R902, R903, R904, R909, R910, R911, R912, R913: 220R, PX4FMUv2.4.6:0402-RES
- removed U201, U901: TXS0108QFN20, PX4FMUv2.4.6:QFN20-RGY
- removed U301: 2908-05WB-MG, PX4FMUv2.4.6:MICROSD
- removed U401: MAX3051, PX4FMUv2.4.6:SOT23-8
- removed U501: L3GD20, PX4FMUv2.4.6:L3G4200DH-MAN
- removed U502: L3GD20H, PX4FMUv2.4.6:LGA-16L
- removed U504: LSM303D, PX4FMUv2.4.6:LGA-16L
- removed U702: LT3469, PX4FMUv2.4.6:SOT23-8
- removed U903: 74LVC2G240, PX4FMUv2.4.6:TSSOP8_SOT505-2
- added TP1: i2c1_SCL, PX4FMUv2.4.6:PAD.04X.04, F.Cu at (137.9, 80.7)
- added TP2: i2c1_SDA, PX4FMUv2.4.6:PAD.04X.04, F.Cu at (139.2, 80.7)
- J901: moved to F.Cu
- moved J901 19.5 mm to (97.8, 104.1), turned to 180 degrees
Connections:
- ADC_PR1 pad P$1: PRESSURE_SENS_IN -> (no net)
- CAN_H1 pad P$1: CAN_H -> (no net)
- CAN_L1 pad P$1: CAN_L -> (no net)
- J301 pad ID: Net-(J301-PadID) -> (no net)
- J901 pad 1: Net-(J901-Pad1) -> (no net)
- J901 pad 12: GND -> (no net)
- J901 pad 15: GND -> (no net)
- J901 pad 18: GND -> (no net)
- J901 pad 21: GND -> (no net)
- J901 pad 24: GND -> (no net)
- J901 pad 27: GND -> (no net)
- J901 pad 3: GND -> (no net)
- J901 pad 30: GND -> (no net)
- J901 pad 31: Net-(J901-Pad31) -> (no net)
- J901 pad 33: GND -> (no net)
- J901 pad 34: Net-(J901-Pad34) -> (no net)
- J901 pad 36: GND -> (no net)
- J901 pad 37: Net-(J901-Pad37) -> (no net)
- J901 pad 39: GND -> (no net)
- J901 pad 4: Net-(J901-Pad4) -> (no net)
- J901 pad 40: Net-(J901-Pad40) -> (no net)
- J901 pad 42: GND -> (no net)
- J901 pad 43: Net-(J901-Pad43) -> (no net)
- J901 pad 45: GND -> (no net)
- J901 pad 46: Net-(J901-Pad46) -> (no net)
- J901 pad 48: GND -> (no net)
- J901 pad 6: GND -> (no net)
- J901 pad 9: GND -> (no net)
- S1RX1 pad P$1: SERIAL1_RX -> (no net)
- S1TX1 pad P$1: SERIAL1_TX -> (no net)
- S2RX1 pad P$1: SERIAL2_RX -> (no net)
- S2TX1 pad P$1: SERIAL2_TX -> (no net)
- U101 pad 1: SPI_EXT_SCK -> (no net)
- U101 pad 16: Net-(U101-Pad16) -> (no net)
- U101 pad 18: FMU_AUX_ADC1 -> (no net)
- U101 pad 3: ~SPI_EXT_NSS -> (no net)
- U101 pad 33: FMU_AUX_ADC2 -> (no net)
- U101 pad 34: PRESSURE_SENS -> (no net)
- U101 pad 4: SPI_EXT_MISO -> (no net)
- U101 pad 40: FMU-CH4 -> (no net)
- U101 pad 42: FMU-CH3 -> (no net)
- U101 pad 44: FMU-CH2 -> (no net)
- U101 pad 45: FMU-CH1 -> (no net)
- U101 pad 5: SPI_EXT_MOSI -> (no net)
- U101 pad 55: FMU-USART3_TX -> (no net)
- U101 pad 56: FMU-USART3_RX -> (no net)
- U101 pad 58: FMU-USART3_CTS -> (no net)
- U101 pad 59: FMU-USART3_RTS -> (no net)
- U101 pad 60: FMU-CH5 -> (no net)
- U101 pad 61: FMU-CH6 -> (no net)
- U101 pad 65: SDIO_D0 -> (no net)
- U101 pad 66: SDIO_D1 -> (no net)
- U101 pad 72: FMU-SWDIO -> (no net)
- U101 pad 76: FMU-SWCLK -> (no net)
- U101 pad 77: ALARM -> (no net)
- U101 pad 78: SDIO_D2 -> (no net)
- U101 pad 79: SDIO_D3 -> (no net)
- U101 pad 8: GPIO_EXT_1 -> (no net)
- U101 pad 80: SDIO_CK -> (no net)
- U101 pad 81: CAN1_RX -> (no net)
- U101 pad 82: CAN1_TX -> (no net)
- U101 pad 83: SDIO_CMD -> (no net)
- U101 pad 84: FMU-USART2_CTS -> (no net)
- U101 pad 85: FMU-USART2_RTS -> (no net)
- U101 pad 86: FMU-USART2_TX -> (no net)
- U101 pad 87: FMU-USART2_RX -> (no net)
- U101 pad 89: FMU-SWO -> (no net)
- U1101 pad P$11: Net-(U1101-PadP$11) -> (no net)
- U1101 pad P$22: Net-(U1101-PadP$22) -> (no net)
- U1101 pad P$23: Net-(U1101-PadP$23) -> (no net)
- U202 pad 1: Net-(U202-Pad1) -> (no net)
- U202 pad 18: Net-(U202-Pad18) -> (no net)
- U202 pad 20: Net-(U202-Pad20) -> (no net)
- U202 pad 3: Net-(U202-Pad3) -> (no net)
- U505 pad 11: Net-(U505-Pad11) -> (no net)
- U505 pad 14: Net-(U505-Pad14) -> (no net)
- U505 pad 15: Net-(U505-Pad15) -> (no net)
- U505 pad 16: Net-(U505-Pad16) -> (no net)
- U505 pad 17: Net-(U505-Pad17) -> (no net)
- U505 pad 19: Net-(U505-Pad19) -> (no net)
- U505 pad 2: Net-(U505-Pad2) -> (no net)
- U505 pad 21: Net-(U505-Pad21) -> (no net)
- U505 pad 22: Net-(U505-Pad22) -> (no net)
- U505 pad 3: Net-(U505-Pad3) -> (no net)
- U505 pad 4: Net-(U505-Pad4) -> (no net)
- U505 pad 5: Net-(U505-Pad5) -> (no net)
- U505 pad 6: Net-(U505-Pad6) -> (no net)
- U505 pad 7: Net-(U505-Pad7) -> (no net)
- U506 pad 4: Net-(U506-Pad4) -> (no net)
- U801 pad 21: SBUS_OUTPUT -> (no net)
- U801 pad 22: SBUS_INPUT -> (no net)
- U801 pad 25: Net-(U801-Pad25) -> (no net)
- U801 pad 26: ~IO-LED_SAFETY -> (no net)
- U801 pad 29: PPM_INPUT -> (no net)
- U801 pad 3: Net-(U801-Pad3) -> (no net)
- U801 pad 32: Net-(U801-Pad32) -> (no net)
- U801 pad 34: /PX4FMUv2.4.6_8/IO-SWDIO -> (no net)
- U801 pad 37: /PX4FMUv2.4.6_8/IO-SWCLK -> (no net)
- U801 pad 39: /PX4FMUv2.4.6_8/IO-SWO -> (no net)
- U801 pad 4: Net-(U801-Pad4) -> (no net)
- U801 pad 40: ~SBUS_OUTPUT_EN -> (no net)
- U801 pad 41: SAFETY -> (no net)
- U801 pad 42: Net-(U801-Pad42) -> (no net)
- U801 pad 43: Net-(U801-Pad43) -> (no net)
Routing:
- net GND: track 280.1 -> 0.00 mm, vias 92 -> 0
- net FMU-VDD_3V3: track 105.4 -> 0.00 mm, vias 17 -> 0
- net VDD_5V_IN: track 96.0 -> 0.00 mm, vias 19 -> 0
- net VBUS: track 65.3 -> 0.00 mm, vias 8 -> 0
- net SPI_INT_MOSI: track 58.3 -> 0.00 mm, vias 6 -> 0
- net SPI_INT_MISO: track 58.3 -> 0.00 mm, vias 6 -> 0
- net SPI_INT_SCK: track 57.5 -> 0.00 mm, vias 6 -> 0
- net ~VDD_BRICK_VALID: track 56.9 -> 0.00 mm, vias 5 -> 0
- net FMU-~RESET: track 56.5 -> 0.00 mm, vias 6 -> 0
- net ~VDD_SERVO_VALID: track 55.3 -> 0.00 mm, vias 5 -> 0
- net ACCEL_DRDY: track 55.1 -> 0.00 mm, vias 4 -> 0
- net /PX4FMUv2.4.6_8/IO-USART1_RX: track 53.0 -> 0.00 mm, vias 5 -> 0
- net ~GYRO_CS: track 52.5 -> 0.00 mm, vias 5 -> 0
- net ~ACCEL_MAG_CS: track 49.8 -> 0.00 mm, vias 4 -> 0
- net ~MPU_CS: track 49.4 -> 0.00 mm, vias 5 -> 0
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- removed copper zone on B.Cu, net VDD_SERVO
