File: PX4FMUv2.4.6_12.sch (KiCad schematic (older format))
At the start: 33 parts, among them M3_MOUNT1101 MOUNT-HOLE3.1MM, M3_MOUNT1102 MOUNT-HOLE3.1MM, M3_MOUNT1103 MOUNT-HOLE3.1MM, M3_MOUNT1104 MOUNT-HOLE3.1MM

Commit message: removed some things
Changed lines of the file:
@@
 EESchema Schematic File Version 4
+LIBS:PX4FMUv2.4.6-cache
 EELAYER 26 0
 EELAYER END
 $Descr User 11818 8333
 encoding utf-8
-Sheet 1 13
+Sheet 13 13
 Title ""
 Date ""
@@
 Parts:\nResistors: 0402 / 1% unless specified otherwise\nCapacitors: 0402 to 1206, ceramic, voltage rating: 10V unless specified
 Wire Notes Line
-	4900 1300 6500 1300
-Wire Notes Line
-	10900 1300 10900 4100
-Wire Notes Line
 	10900 4100 8800 4100
 Wire Notes Line
-	8800 4100 8800 3300
-Wire Notes Line
-	8800 3300 8800 1300
-Wire Notes Line
-	8800 1300 6500 1300
-Wire Notes Line
-	6500 1300 6500 3300
-Wire Notes Line
-	6500 3300 6500 5900
-Wire Notes Line
 	6500 5900 4900 5900
 Wire Notes Line
-	4900 5900 4900 1300
-Wire Notes Line
 	6500 3300 8800 3300
-Wire Notes Line
-	4900 1300 4900 1000
-Wire Notes Line
-	4900 1000 6500 1000
-Wire Notes Line
-	8800 1000 10900 1000
-Wire Notes Line
-	10900 1000 10900 1300
-Wire Notes Line
-	10900 1300 8800 1300
-Wire Notes Line
-	8800 1300 8800 1000
-Wire Notes Line
-	8800 1000 6500 1000
-Wire Notes Line
-	6500 1000 6500 1300
 Text Notes 5000 1200 0    100  ~ 0
 COMMS
@@
 Text Notes 6600 1200 0    100  ~ 0
 STATUS AND ANALOG
+Wire Notes Line
+	10900 1000 10900 4100
+Wire Notes Line
+	4900 1000 4900 5900
+Wire Notes Line
+	4900 1000 10900 1000
+Wire Notes Line
+	4900 1300 10900 1300
+Wire Notes Line
+	8800 1000 8800 4100
+Wire Notes Line
+	6500 1000 6500 5900
 $EndSCHEMATC

Commit message: removed more things
Parts:
- added TP1: i2c1_SCL, PX4FMUv2.4.6:PAD.04X.04, symbol PX4FMUv2.4.6-eagle-import:PAD.04
- added TP2: i2c1_SDA, PX4FMUv2.4.6:PAD.04X.04, symbol PX4FMUv2.4.6-eagle-import:PAD.04
Connections:
- new net FMU-I2C1_SCL: TP1.P$1
- new net FMU-I2C1_SDA: TP2.P$1
Changed lines of the file:
@@
 Wire Notes Line
 	6500 1000 6500 5900
+Text GLabel 5800 6150 0    50   BiDi ~ 0
+FMU-I2C1_SCL
+Text GLabel 5800 6500 0    50   BiDi ~ 0
+FMU-I2C1_SDA
+Wire Wire Line
+	5800 6150 6000 6150
+Wire Wire Line
+	5800 6500 6000 6500
+$Comp
+L PX4FMUv2.4.6-eagle-import:PAD.04 TP1
+U 1 1 5C20AFF8
+P 6300 6150
+F 0 "TP1" H 6427 6150 42  0000 L CNN
+F 1 "i2c1_SCL" H 6300 6150 50  0001 C CNN
+F 2 "PX4FMUv2.4.6:PAD.04X.04" H 6300 6150 50  0001 C CNN
+F 3 "" H 6300 6150 50  0001 C CNN
+	1    6300 6150
+	1    0    0    -1
+$EndComp
+$Comp
+L PX4FMUv2.4.6-eagle-import:PAD.04 TP2
+U 1 1 5C20B076
+P 6300 6500
+F 0 "TP2" H 6427 6500 42  0000 L CNN
+F 1 "i2c1_SDA" H 6300 6500 50  0001 C CNN
+F 2 "PX4FMUv2.4.6:PAD.04X.04" H 6300 6500 50  0001 C CNN
+F 3 "" H 6300 6500 50  0001 C CNN
+	1    6300 6500
+	1    0    0    -1
+$EndComp
 $EndSCHEMATC
