File: PX4FMUv2.4.6_2.sch (KiCad schematic (older format))
At the start: 23 parts, among them J203 DF13C-6P-1.25V, U201 TXS0108QFN20, U202 TXS0108QFN20

Commit message: removed more things
Parts:
- removed C201: 0u1, PX4FMUv2.4.6:0402-CAP, symbol PX4FMUv2.4.6-eagle-import:CAP0402
- removed R201, R202, R203, R204, R208, R209, R210, R211, R215, R216: 120R, PX4FMUv2.4.6:0402-RES, symbol PX4FMUv2.4.6-eagle-import:RESISTOR0402-RES
- removed U201: TXS0108QFN20, PX4FMUv2.4.6:QFN20-RGY, symbol PX4FMUv2.4.6-eagle-import:TXS0108QFN20
