File: PX4FMUv2.4.6_3.sch (KiCad schematic (older format))
At the start: 12 parts, among them J301 47346-0001, J302 DF13C-4P-1.25V, U301 2908-05WB-MG, U302 NUF2042XV6

Commit message: removed some things
Parts:
- removed J302: DF13C-4P-1.25V, PX4FMUv2.4.6:DF13C-4P-1.25V, symbol PX4FMUv2.4.6-eagle-import:DF13-4P-1.25V
- removed R301, R302, R303, R304, R305: 100K, PX4FMUv2.4.6:0402-RES, symbol PX4FMUv2.4.6-eagle-import:RESISTOR0402-RES
- removed U301: 2908-05WB-MG, PX4FMUv2.4.6:MICROSD, symbol PX4FMUv2.4.6-eagle-import:MICROSDSDI
Other:
- note removed: "To be used with panel-\nmount micro USB connectors:\n - Amphenol MUSBK15230"
- note removed: "microSD"
Changed lines of the file:
@@
 EESchema Schematic File Version 4
+LIBS:PX4FMUv2.4.6-cache
 EELAYER 26 0
 EELAYER END
@@
 FMU-SWDIO
 Wire Wire Line
-	4200 1200 3900 1200
-Wire Wire Line
-	3900 1200 3900 2500
-Wire Wire Line
-	4200 2500 3900 2500
-Wire Wire Line
-	3900 1200 3000 1200
-Wire Wire Line
 	3000 1200 3000 1300
 Wire Wire Line
@@
 Text GLabel 2200 1300 0    50   BiDi ~ 0
 VBUS
-Connection ~ 3900 1200
 Connection ~ 3000 1300
 Wire Wire Line
@@
 	4200 1900 4100 1900
 Wire Wire Line
-	4100 1900 4100 2800
-Wire Wire Line
-	4100 2800 4100 2900
-Wire Wire Line
 	4100 2900 4100 3000
 Wire Wire Line
 	4200 1600 4200 1900
-Wire Wire Line
-	4200 2800 4100 2800
 Wire Wire Line
 	3000 2600 3000 2900
@@
 Connection ~ 4450 1900
 Connection ~ 4550 1900
-Connection ~ 4100 2800
 Connection ~ 4100 2900
 Text GLabel 4650 1900 0    10   BiDi ~ 0
@@
 GND
 Wire Wire Line
-	4000 5400 4000 5100
-Wire Wire Line
-	4000 5100 4100 5100
-Text GLabel 4000 5400 0    10   BiDi ~ 0
-GND
-Wire Wire Line
 	9700 5000 9200 5000
 Text GLabel 9200 5000 0    50   BiDi ~ 0
 FMU-VDD_3V3
-Wire Wire Line
-	4100 4400 4000 4400
-Wire Wire Line
-	4000 4400 4000 3800
-Wire Wire Line
-	2500 3800 2600 3800
-Wire Wire Line
-	2600 3800 2600 3900
-Wire Wire Line
-	2600 3800 2900 3800
-Wire Wire Line
-	2900 3800 2900 3900
-Wire Wire Line
-	2900 3800 3200 3800
-Wire Wire Line
-	3200 3800 3200 3900
-Wire Wire Line
-	3200 3800 3500 3800
-Wire Wire Line
-	3500 3800 3500 3900
-Wire Wire Line
-	3500 3800 3800 3800
-Wire Wire Line
-	3800 3800 3800 3900
-Wire Wire Line
-	3800 3800 4000 3800
-Text GLabel 2500 3800 0    50   BiDi ~ 0
-FMU-VDD_3V3
-Connection ~ 2600 3800
-Connection ~ 2900 3800
-Connection ~ 3200 3800
-Connection ~ 3500 3800
-Connection ~ 3800 3800
 Wire Wire Line
 	6600 1200 6800 1200
@@
 	3800 1300 4200 1300
 Wire Wire Line
-	4200 2700 3800 2700
-Wire Wire Line
-	3800 2700 3800 2200
-Wire Wire Line
 	3800 2200 3800 1300
 Wire Wire Line
 	3500 2200 3800 2200
-Connection ~ 3800 2200
 Wire Wire Line
 	3700 1400 4200 1400
 Wire Wire Line
-	4200 2600 3700 2600
-Wire Wire Line
-	3700 2600 3700 1800
-Wire Wire Line
 	3700 1800 3700 1400
 Wire Wire Line
 	3500 1800 3700 1800
-Connection ~ 3700 1800
 Wire Wire Line
 	2500 1800 2200 1800
@@
 Text GLabel 2200 2200 0    50   BiDi ~ 0
 OTG_FS_DM
-Wire Wire Line
-	4100 4900 3500 4900
-Wire Wire Line
-	3500 4900 2500 4900
-Wire Wire Line
-	3500 4300 3500 4900
-Text GLabel 2500 4900 0    50   BiDi ~ 0
-SDIO_D0
-Connection ~ 3500 4900
-Wire Wire Line
-	4100 5000 3800 5000
-Wire Wire Line
-	3800 5000 2500 5000
-Wire Wire Line
-	3800 4300 3800 5000
-Text GLabel 2500 5000 0    50   BiDi ~ 0
-SDIO_D1
-Connection ~ 3800 5000
-Wire Wire Line
-	4100 4600 2600 4600
-Wire Wire Line
-	2600 4600 2500 4600
-Wire Wire Line
-	2600 4300 2600 4600
-Text GLabel 2500 4600 0    50   BiDi ~ 0
-SDIO_D2
-Connection ~ 2600 4600
-Wire Wire Line
-	4100 4700 2900 4700
-Wire Wire Line
-	2900 4700 2500 4700
-Wire Wire Line
-	2900 4300 2900 4700
-Text GLabel 2500 4700 0    50   BiDi ~ 0
-SDIO_D3
-Connection ~ 2900 4700
-Wire Wire Line
-	4100 4500 2500 4500
-Text GLabel 2500 4500 0    50   BiDi ~ 0
-SDIO_CK
-Wire Wire Line
-	4100 4800 3200 4800
-Wire Wire Line
-	3200 4800 2500 4800
-Wire Wire Line
-	3200 4300 3200 4800
-Text GLabel 2500 4800 0    50   BiDi ~ 0
-SDIO_CMD
-Connection ~ 3200 4800
 Wire Wire Line
 	6800 1800 6700 1800
@@
 F 3 "" H 9800 5500 50  0001 C CNN
 	9    9800 5500
-	1    0    0    -1
-$EndComp
-$Comp
-L PX4FMUv2.4.6-eagle-import:MICROSDSDI U301
-U 1 0 44E587D1B2B37021
-P 4350 4650
-AR Path="/44E587D1B2B37021" Ref="U301"  Part="1"
-AR Path="/5C109013/44E587D1B2B37021" Ref="U301"  Part="1"
-F 0 "U301" H 4200 5000 59  0000 L BNN
-F 1 "2908-05WB-MG" H 4200 4000 59  0000 L BNN
-F 2 "PX4FMUv2.4.6:MICROSD" H 4350 4650 50  0001 C CNN
-F 3 "" H 4350 4650 50  0001 C CNN
-	1    4350 4650
-	1    0    0    -1
-$EndComp
-$Comp
-L PX4FMUv2.4.6-eagle-import:GND #GND20
-U 1 0 1D4613EF2DF12463
-P 4000 5500
-AR Path="/1D4613EF2DF12463" Ref="#GND20"  Part="1"
-AR Path="/5C109013/1D4613EF2DF12463" Ref="#GND020"  Part="1"
-F 0 "#GND020" H 4000 5500 50  0001 C CNN
-F 1 "GND" H 3900 5400 59  0000 L BNN
-F 2 "" H 4000 5500 50  0001 C CNN
-F 3 "" H 4000 5500 50  0001 C CNN
-	1    4000 5500
 	1    0    0    -1
 $EndComp
@@
 $EndComp
 $Comp
-L PX4FMUv2.4.6-eagle-import:RESISTOR0402-RES R301
-U 1 0 F0C0FF184D5C2B5C
-P 2600 4100
-AR Path="/F0C0FF184D5C2B5C" Ref="R301"  Part="1"
-AR Path="/5C109013/F0C0FF184D5C2B5C" Ref="R301"  Part="1"
-F 0 "R301" H 2450 4159 59  0000 L BNN
-F 1 "100K" H 2450 3970 59  0000 L BNN
-F 2 "PX4FMUv2.4.6:0402-RES" H 2600 4100 50  0001 C CNN
-F 3 "" H 2600 4100 50  0001 C CNN
-	1    2600 4100
-	0    -1   -1   0
-$EndComp
-$Comp
-L PX4FMUv2.4.6-eagle-import:RESISTOR0402-RES R302
-U 1 0 53282B10B39218E6
-P 2900 4100
-AR Path="/53282B10B39218E6" Ref="R302"  Part="1"
-AR Path="/5C109013/53282B10B39218E6" Ref="R302"  Part="1"
-F 0 "R302" H 2750 4159 59  0000 L BNN
-F 1 "100K" H 2750 3970 59  0000 L BNN
-F 2 "PX4FMUv2.4.6:0402-RES" H 2900 4100 50  0001 C CNN
-F 3 "" H 2900 4100 50  0001 C CNN
-	1    2900 4100
-	0    -1   -1   0
-$EndComp
-$Comp
-L PX4FMUv2.4.6-eagle-import:RESISTOR0402-RES R303
-U 1 0 D9D6447F6560EC56
-P 3200 4100
-AR Path="/D9D6447F6560EC56" Ref="R303"  Part="1"
-AR Path="/5C109013/D9D6447F6560EC56" Ref="R303"  Part="1"
-F 0 "R303" H 3050 4159 59  0000 L BNN
-F 1 "100K" H 3050 3970 59  0000 L BNN
-F 2 "PX4FMUv2.4.6:0402-RES" H 3200 4100 50  0001 C CNN
-F 3 "" H 3200 4100 50  0001 C CNN
-	1    3200 4100
-	0    -1   -1   0
-$EndComp
-$Comp
-L PX4FMUv2.4.6-eagle-import:RESISTOR0402-RES R304
-U 1 0 9C2F127629F7151B
-P 3500 4100
-AR Path="/9C2F127629F7151B" Ref="R304"  Part="1"
-AR Path="/5C109013/9C2F127629F7151B" Ref="R304"  Part="1"
-F 0 "R304" H 3350 4159 59  0000 L BNN
-F 1 "100K" H 3350 3970 59  0000 L BNN
-F 2 "PX4FMUv2.4.6:0402-RES" H 3500 4100 50  0001 C CNN
-F 3 "" H 3500 4100 50  0001 C CNN
-	1    3500 4100
-	0    -1   -1   0
-$EndComp
-$Comp
-L PX4FMUv2.4.6-eagle-import:RESISTOR0402-RES R305
-U 1 0 7FC7153AA04D91FB
-P 3800 4100
-AR Path="/7FC7153AA04D91FB" Ref="R305"  Part="1"
-AR Path="/5C109013/7FC7153AA04D91FB" Ref="R305"  Part="1"
-F 0 "R305" H 3650 4159 59  0000 L BNN
-F 1 "100K" H 3650 3970 59  0000 L BNN
-F 2 "PX4FMUv2.4.6:0402-RES" H 3800 4100 50  0001 C CNN
-F 3 "" H 3800 4100 50  0001 C CNN
-	1    3800 4100
-	0    -1   -1   0
-$EndComp
-$Comp
-L PX4FMUv2.4.6-eagle-import:DF13-4P-1.25V J302
-U 1 0 FAB04A95DB771C7E
-P 4400 2600
-AR Path="/FAB04A95DB771C7E" Ref="J302"  Part="1"
-AR Path="/5C109013/FAB04A95DB771C7E" Ref="J302"  Part="1"
-F 0 "J302" H 4325 2800 59  0000 L BNN
-F 1 "DF13C-4P-1.25V" H 4325 2238 59  0000 L BNN
-F 2 "PX4FMUv2.4.6:DF13C-4P-1.25V" H 4400 2600 50  0001 C CNN
-F 3 "" H 4400 2600 50  0001 C CNN
-	1    4400 2600
-	1    0    0    -1
-$EndComp
-$Comp
 L PX4FMUv2.4.6-eagle-import:NUF2042XV6 U302
 U 1 0 EC9C0E2A40595D8A
@@
 Text Notes 7300 6700 0    73   ~ 0
 USB\nmicroSD\nExpansion
-Text Notes 4200 5400 0    59   ~ 0
-microSD
-Text Notes 4600 2800 0    47   ~ 0
-To be used with panel-\nmount micro USB connectors:\n - Amphenol MUSBK15230
+Wire Wire Line
+	4100 1900 4100 2900
+Wire Wire Line
+	3000 1200 4200 1200
 $EndSCHEMATC

Commit message: removed more things
Parts:
- removed JX301: ARM_MINI_JTAG-SMT, PX4FMUv2.4.6:FTSH-105-01-XXX-DV-K, symbol PX4FMUv2.4.6-eagle-import:ARM_MINI_JTAG-SMT
Changed lines of the file:
@@
 $EndDescr
-Wire Wire Line
-	9700 5100 9200 5100
-Text GLabel 9200 5100 0    50   BiDi ~ 0
-FMU-SWDIO
 Wire Wire Line
 	3000 1200 3000 1300
@@
 Text GLabel 4650 1900 0    10   BiDi ~ 0
 GND
-Wire Wire Line
-	9700 5600 9500 5600
-Wire Wire Line
-	9500 5600 9500 5700
-Wire Wire Line
-	9500 5700 9500 5800
-Wire Wire Line
-	9500 5800 9500 5900
-Wire Wire Line
-	9700 5700 9500 5700
-Wire Wire Line
-	9500 5800 9700 5800
-Connection ~ 9500 5700
-Connection ~ 9500 5800
-Text GLabel 9700 5600 0    10   BiDi ~ 0
-GND
-Wire Wire Line
-	9700 5000 9200 5000
-Text GLabel 9200 5000 0    50   BiDi ~ 0
-FMU-VDD_3V3
 Wire Wire Line
 	6600 1200 6800 1200
@@
 Text GLabel 6700 1900 0    50   BiDi ~ 0
 FMU-I2C2_SDA
-Wire Wire Line
-	9700 5300 9200 5300
-Text GLabel 9200 5300 0    50   BiDi ~ 0
-FMU-SWO
-Wire Wire Line
-	9700 5200 9200 5200
-Text GLabel 9200 5200 0    50   BiDi ~ 0
-FMU-SWCLK
 $Comp
 L PX4FMUv2.4.6-eagle-import:A4L-LOC #FRAME6
@@
 	1    0    0    -1
 $EndComp
-$Comp
-L PX4FMUv2.4.6-eagle-import:GND #GND16
-U 1 0 8316678299D4D269
-P 9500 6000
-AR Path="/8316678299D4D269" Ref="#GND16"  Part="1"
-AR Path="/5C109013/8316678299D4D269" Ref="#GND016"  Part="1"
-F 0 "#GND016" H 9500 6000 50  0001 C CNN
-F 1 "GND" H 9400 5900 59  0000 L BNN
-F 2 "" H 9500 6000 50  0001 C CNN
-F 3 "" H 9500 6000 50  0001 C CNN
-	1    9500 6000
-	1    0    0    -1
-$EndComp
-$Comp
-L PX4FMUv2.4.6-eagle-import:ARM_MINI_JTAG-SMT JX301
-U 1 0 F99DB6D9CEB5AE7F
-P 9800 5000
-AR Path="/F99DB6D9CEB5AE7F" Ref="JX301"  Part="1"
-AR Path="/5C109013/F99DB6D9CEB5AE7F" Ref="JX301"  Part="1"
-F 0 "JX301" H 9900 4970 51  0000 L BNN
-F 1 "ARM_MINI_JTAG-SMT" H 9770 5055 59  0001 L BNN
-F 2 "PX4FMUv2.4.6:FTSH-105-01-XXX-DV-K" H 9800 5000 50  0001 C CNN
-F 3 "" H 9800 5000 50  0001 C CNN
-	1    9800 5000
-	1    0    0    -1
-$EndComp
-$Comp
-L PX4FMUv2.4.6-eagle-import:ARM_MINI_JTAG-SMT JX301
-U 2 0 F99DB6D9CEB5AE73
-P 9800 5100
-AR Path="/F99DB6D9CEB5AE73" Ref="JX301"  Part="2"
-AR Path="/5C109013/F99DB6D9CEB5AE73" Ref="JX301"  Part="2"
-F 0 "JX301" H 9900 5070 51  0000 L BNN
-F 1 "ARM_MINI_JTAG-SMT" H 9770 5155 59  0001 L BNN
-F 2 "PX4FMUv2.4.6:FTSH-105-01-XXX-DV-K" H 9800 5100 50  0001 C CNN
-F 3 "" H 9800 5100 50  0001 C CNN
-	2    9800 5100
-	1    0    0    -1
-$EndComp
-$Comp
-L PX4FMUv2.4.6-eagle-import:ARM_MINI_JTAG-SMT JX301
-U 3 0 F99DB6D9CEB5AE77
-P 9800 5600
-AR Path="/F99DB6D9CEB5AE77" Ref="JX301"  Part="3"
-AR Path="/5C109013/F99DB6D9CEB5AE77" Ref="JX301"  Part="3"
-F 0 "JX301" H 9900 5570 51  0000 L BNN
-F 1 "ARM_MINI_JTAG-SMT" H 9770 5655 59  0001 L BNN
-F 2 "PX4FMUv2.4.6:FTSH-105-01-XXX-DV-K" H 9800 5600 50  0001 C CNN
-F 3 "" H 9800 5600 50  0001 C CNN
-	3    9800 5600
-	1    0    0    -1
-$EndComp
-$Comp
-L PX4FMUv2.4.6-eagle-import:ARM_MINI_JTAG-SMT JX301
-U 4 0 F99DB6D9CEB5AE6B
-P 9800 5200
-AR Path="/F99DB6D9CEB5AE6B" Ref="JX301"  Part="4"
-AR Path="/5C109013/F99DB6D9CEB5AE6B" Ref="JX301"  Part="4"
-F 0 "JX301" H 9900 5170 51  0000 L BNN
-F 1 "ARM_MINI_JTAG-SMT" H 9770 5255 59  0001 L BNN
-F 2 "PX4FMUv2.4.6:FTSH-105-01-XXX-DV-K" H 9800 5200 50  0001 C CNN
-F 3 "" H 9800 5200 50  0001 C CNN
-	4    9800 5200
-	1    0    0    -1
-$EndComp
-$Comp
-L PX4FMUv2.4.6-eagle-import:ARM_MINI_JTAG-SMT JX301
-U 5 0 F99DB6D9CEB5AE6F
-P 9800 5700
-AR Path="/F99DB6D9CEB5AE6F" Ref="JX301"  Part="5"
-AR Path="/5C109013/F99DB6D9CEB5AE6F" Ref="JX301"  Part="5"
-F 0 "JX301" H 9900 5670 51  0000 L BNN
-F 1 "ARM_MINI_JTAG-SMT" H 9770 5755 59  0001 L BNN
-F 2 "PX4FMUv2.4.6:FTSH-105-01-XXX-DV-K" H 9800 5700 50  0001 C CNN
-F 3 "" H 9800 5700 50  0001 C CNN
-	5    9800 5700
-	1    0    0    -1
-$EndComp
-$Comp
-L PX4FMUv2.4.6-eagle-import:ARM_MINI_JTAG-SMT JX301
-U 6 0 F99DB6D9CEB5AE63
-P 9800 5300
-AR Path="/F99DB6D9CEB5AE63" Ref="JX301"  Part="6"
-AR Path="/5C109013/F99DB6D9CEB5AE63" Ref="JX301"  Part="6"
-F 0 "JX301" H 9900 5270 51  0000 L BNN
-F 1 "ARM_MINI_JTAG-SMT" H 9770 5355 59  0001 L BNN
-F 2 "PX4FMUv2.4.6:FTSH-105-01-XXX-DV-K" H 9800 5300 50  0001 C CNN
-F 3 "" H 9800 5300 50  0001 C CNN
-	6    9800 5300
-	1    0    0    -1
-$EndComp
-$Comp
-L PX4FMUv2.4.6-eagle-import:ARM_MINI_JTAG-SMT JX301
-U 7 0 F99DB6D9CEB5AE67
-P 9800 5400
-AR Path="/F99DB6D9CEB5AE67" Ref="JX301"  Part="7"
-AR Path="/5C109013/F99DB6D9CEB5AE67" Ref="JX301"  Part="7"
-F 0 "JX301" H 9900 5370 51  0000 L BNN
-F 1 "ARM_MINI_JTAG-SMT" H 9770 5455 59  0001 L BNN
-F 2 "PX4FMUv2.4.6:FTSH-105-01-XXX-DV-K" H 9800 5400 50  0001 C CNN
-F 3 "" H 9800 5400 50  0001 C CNN
-	7    9800 5400
-	1    0    0    -1
-$EndComp
-$Comp
-L PX4FMUv2.4.6-eagle-import:ARM_MINI_JTAG-SMT JX301
-U 8 0 F99DB6D9CEB5AE5B
-P 9800 5800
-AR Path="/F99DB6D9CEB5AE5B" Ref="JX301"  Part="8"
-AR Path="/5C109013/F99DB6D9CEB5AE5B" Ref="JX301"  Part="8"
-F 0 "JX301" H 9900 5770 51  0000 L BNN
-F 1 "ARM_MINI_JTAG-SMT" H 9770 5855 59  0001 L BNN
-F 2 "PX4FMUv2.4.6:FTSH-105-01-XXX-DV-K" H 9800 5800 50  0001 C CNN
-F 3 "" H 9800 5800 50  0001 C CNN
-	8    9800 5800
-	1    0    0    -1
-$EndComp
-$Comp
-L PX4FMUv2.4.6-eagle-import:ARM_MINI_JTAG-SMT JX301
-U 9 0 F99DB6D9CEB5AE5F
-P 9800 5500
-AR Path="/F99DB6D9CEB5AE5F" Ref="JX301"  Part="9"
-AR Path="/5C109013/F99DB6D9CEB5AE5F" Ref="JX301"  Part="9"
-F 0 "JX301" H 9900 5470 51  0000 L BNN
-F 1 "ARM_MINI_JTAG-SMT" H 9770 5555 59  0001 L BNN
-F 2 "PX4FMUv2.4.6:FTSH-105-01-XXX-DV-K" H 9800 5500 50  0001 C CNN
-F 3 "" H 9800 5500 50  0001 C CNN
-	9    9800 5500
-	1    0    0    -1
-$EndComp
