File: PX4FMUv2.4.6_8.sch (KiCad schematic (older format))
At the start: 17 parts, among them J801 JST-ZH-3, U801 STM32F10XCXT6, X801 3.2x2.5 mm / 24 MHz / 15 ppm

Commit message: removed more things
Parts:
- removed JX801: HEADER-3X1BOARDEDGE-SHORT, PX4FMUv2.4.6:HEADER_3X01_SMD_H_BOARD_EDGE_SHORT, symbol PX4FMUv2.4.6-eagle-import:HEADER-3X1BOARDEDGE-SHORT
- removed JX802: ARM_MINI_JTAG-SMT, PX4FMUv2.4.6:FTSH-105-01-XXX-DV-K, symbol PX4FMUv2.4.6-eagle-import:ARM_MINI_JTAG-SMT
Other:
- note removed: "IO_SERIAL1"
Changed lines of the file:
@@
-GND
-Wire Wire Line
-	9700 6100 9700 6000
-Wire Wire Line
-	9700 6000 9700 5900
-Wire Wire Line
-	9700 5900 9900 5900
-Wire Wire Line
-	9900 6000 9700 6000
-Wire Wire Line
-	9700 6100 9900 6100
-Wire Wire Line
-	9700 6200 9700 6100
-Connection ~ 9700 6000
-Connection ~ 9700 6100
-Text GLabel 9700 6100 0    10   BiDi ~ 0
 GND
 Wire Wire Line
@@
 GND
 Wire Wire Line
-	5900 1400 5900 1300
-Wire Wire Line
-	5900 1300 6000 1300
-Text GLabel 5900 1400 0    10   BiDi ~ 0
-GND
-Wire Wire Line
 	2000 2200 2300 2200
 Text Label 2300 2200 0    50   ~ 0
-IO-USART1_RX
-Wire Wire Line
-	6000 1200 5800 1200
-Text Label 5800 1200 2    50   ~ 0
 IO-USART1_RX
 Wire Wire Line
@@
 IO-VDD_3V3
 Wire Wire Line
-	9900 5200 9700 5200
-Text GLabel 9700 5200 0    50   BiDi ~ 0
-IO-VDD_3V3
-Wire Wire Line
 	9800 4100 9700 4100
 Wire Wire Line
@@
 IO-USART1_TX
 Wire Wire Line
-	6000 1100 5800 1100
-Text GLabel 5800 1100 0    50   BiDi ~ 0
-IO-USART1_TX
-Wire Wire Line
 	2000 3600 2300 3600
 Text GLabel 2300 3600 2    50   BiDi ~ 0
@@
 IO-SWDIO
 Wire Wire Line
-	9700 5300 9900 5300
-Text Label 9700 5300 2    50   ~ 0
-IO-SWDIO
-Wire Wire Line
 	2000 2600 2300 2600
 Text Label 2300 2600 0    50   ~ 0
 IO-SWCLK
 Wire Wire Line
-	9900 5400 9700 5400
-Text Label 9700 5400 2    50   ~ 0
-IO-SWCLK
-Wire Wire Line
 	3700 900  3800 900
 Text GLabel 3800 900  2    50   BiDi ~ 0
@@
 	2000 3400 2300 3400
 Text Label 2300 3400 0    50   ~ 0
-IO-SWO
-Wire Wire Line
-	9900 5500 9700 5500
-Text Label 9700 5500 2    50   ~ 0
 IO-SWO
 Wire Wire Line
@@
 $EndComp
 $Comp
-L PX4FMUv2.4.6-eagle-import:ARM_MINI_JTAG-SMT JX802
-U 1 0 743F0D129647417E
-P 10000 5200
-AR Path="/743F0D129647417E" Ref="JX802"  Part="1"
-AR Path="/5C109CCF/743F0D129647417E" Ref="JX802"  Part="1"
-F 0 "JX802" H 10100 5170 51  0000 L BNN
-F 1 "ARM_MINI_JTAG-SMT" H 9670 5255 59  0001 L BNN
-F 2 "PX4FMUv2.4.6:FTSH-105-01-XXX-DV-K" H 10000 5200 50  0001 C CNN
-F 3 "" H 10000 5200 50  0001 C CNN
-	1    10000 5200
-	1    0    0    -1
-$EndComp
-$Comp
-L PX4FMUv2.4.6-eagle-import:ARM_MINI_JTAG-SMT JX802
-U 2 0 743F0D1296474172
-P 10000 5300
-AR Path="/743F0D1296474172" Ref="JX802"  Part="2"
-AR Path="/5C109CCF/743F0D1296474172" Ref="JX802"  Part="2"
-F 0 "JX802" H 10100 5270 51  0000 L BNN
-F 1 "ARM_MINI_JTAG-SMT" H 9970 5355 59  0001 L BNN
-F 2 "PX4FMUv2.4.6:FTSH-105-01-XXX-DV-K" H 10000 5300 50  0001 C CNN
-F 3 "" H 10000 5300 50  0001 C CNN
-	2    10000 5300
-	1    0    0    -1
-$EndComp
-$Comp
-L PX4FMUv2.4.6-eagle-import:ARM_MINI_JTAG-SMT JX802
-U 3 0 743F0D1296474176
-P 10000 5900
-AR Path="/743F0D1296474176" Ref="JX802"  Part="3"
-AR Path="/5C109CCF/743F0D1296474176" Ref="JX802"  Part="3"
-F 0 "JX802" H 10100 5870 51  0000 L BNN
-F 1 "ARM_MINI_JTAG-SMT" H 9970 5955 59  0001 L BNN
-F 2 "PX4FMUv2.4.6:FTSH-105-01-XXX-DV-K" H 10000 5900 50  0001 C CNN
-F 3 "" H 10000 5900 50  0001 C CNN
-	3    10000 5900
-	1    0    0    -1
-$EndComp
-$Comp
-L PX4FMUv2.4.6-eagle-import:ARM_MINI_JTAG-SMT JX802
-U 4 0 743F0D129647416A
-P 10000 5400
-AR Path="/743F0D129647416A" Ref="JX802"  Part="4"
-AR Path="/5C109CCF/743F0D129647416A" Ref="JX802"  Part="4"
-F 0 "JX802" H 10100 5370 51  0000 L BNN
-F 1 "ARM_MINI_JTAG-SMT" H 9970 5455 59  0001 L BNN
-F 2 "PX4FMUv2.4.6:FTSH-105-01-XXX-DV-K" H 10000 5400 50  0001 C CNN
-F 3 "" H 10000 5400 50  0001 C CNN
-	4    10000 5400
-	1    0    0    -1
-$EndComp
-$Comp
-L PX4FMUv2.4.6-eagle-import:ARM_MINI_JTAG-SMT JX802
-U 5 0 743F0D129647416E
-P 10000 6000
-AR Path="/743F0D129647416E" Ref="JX802"  Part="5"
-AR Path="/5C109CCF/743F0D129647416E" Ref="JX802"  Part="5"
-F 0 "JX802" H 10100 5970 51  0000 L BNN
-F 1 "ARM_MINI_JTAG-SMT" H 9970 6055 59  0001 L BNN
-F 2 "PX4FMUv2.4.6:FTSH-105-01-XXX-DV-K" H 10000 6000 50  0001 C CNN
-F 3 "" H 10000 6000 50  0001 C CNN
-	5    10000 6000
-	1    0    0    -1
-$EndComp
-$Comp
-L PX4FMUv2.4.6-eagle-import:ARM_MINI_JTAG-SMT JX802
-U 6 0 743F0D1296474162
-P 10000 5500
-AR Path="/743F0D1296474162" Ref="JX802"  Part="6"
-AR Path="/5C109CCF/743F0D1296474162" Ref="JX802"  Part="6"
-F 0 "JX802" H 10100 5470 51  0000 L BNN
-F 1 "ARM_MINI_JTAG-SMT" H 9970 5555 59  0001 L BNN
-F 2 "PX4FMUv2.4.6:FTSH-105-01-XXX-DV-K" H 10000 5500 50  0001 C CNN
-F 3 "" H 10000 5500 50  0001 C CNN
-	6    10000 5500
-	1    0    0    -1
-$EndComp
-$Comp
-L PX4FMUv2.4.6-eagle-import:ARM_MINI_JTAG-SMT JX802
-U 7 0 743F0D1296474166
-P 10000 5600
-AR Path="/743F0D1296474166" Ref="JX802"  Part="7"
-AR Path="/5C109CCF/743F0D1296474166" Ref="JX802"  Part="7"
-F 0 "JX802" H 10100 5570 51  0000 L BNN
-F 1 "ARM_MINI_JTAG-SMT" H 9970 5655 59  0001 L BNN
-F 2 "PX4FMUv2.4.6:FTSH-105-01-XXX-DV-K" H 10000 5600 50  0001 C CNN
-F 3 "" H 10000 5600 50  0001 C CNN
-	7    10000 5600
-	1    0    0    -1
-$EndComp
-$Comp
-L PX4FMUv2.4.6-eagle-import:ARM_MINI_JTAG-SMT JX802
-U 8 0 743F0D129647415A
-P 10000 6100
-AR Path="/743F0D129647415A" Ref="JX802"  Part="8"
-AR Path="/5C109CCF/743F0D129647415A" Ref="JX802"  Part="8"
-F 0 "JX802" H 10100 6070 51  0000 L BNN
-F 1 "ARM_MINI_JTAG-SMT" H 9970 6155 59  0001 L BNN
-F 2 "PX4FMUv2.4.6:FTSH-105-01-XXX-DV-K" H 10000 6100 50  0001 C CNN
-F 3 "" H 10000 6100 50  0001 C CNN
-	8    10000 6100
-	1    0    0    -1
-$EndComp
-$Comp
-L PX4FMUv2.4.6-eagle-import:ARM_MINI_JTAG-SMT JX802
-U 9 0 743F0D129647415E
-P 10000 5700
-AR Path="/743F0D129647415E" Ref="JX802"  Part="9"
-AR Path="/5C109CCF/743F0D129647415E" Ref="JX802"  Part="9"
-F 0 "JX802" H 10100 5670 51  0000 L BNN
-F 1 "ARM_MINI_JTAG-SMT" H 9970 5755 59  0001 L BNN
-F 2 "PX4FMUv2.4.6:FTSH-105-01-XXX-DV-K" H 10000 5700 50  0001 C CNN
-F 3 "" H 10000 5700 50  0001 C CNN
-	9    10000 5700
-	1    0    0    -1
-$EndComp
-$Comp
-L PX4FMUv2.4.6-eagle-import:GND #GND45
-U 1 0 9FE288429E0B3A99
-P 9700 6300
-AR Path="/9FE288429E0B3A99" Ref="#GND45"  Part="1"
-AR Path="/5C109CCF/9FE288429E0B3A99" Ref="#GND045"  Part="1"
-F 0 "#GND045" H 9700 6300 50  0001 C CNN
-F 1 "GND" H 9600 6200 59  0000 L BNN
-F 2 "" H 9700 6300 50  0001 C CNN
-F 3 "" H 9700 6300 50  0001 C CNN
-	1    9700 6300
-	1    0    0    -1
-$EndComp
-$Comp
 L PX4FMUv2.4.6-eagle-import:GND #GND46
 U 1 0 3045C7A0D2AB3227
@@
 $EndComp
 $Comp
-L PX4FMUv2.4.6-eagle-import:HEADER-3X1BOARDEDGE-SHORT JX801
-U 1 0 6BB659706DA45596
-P 6300 1300
-AR Path="/6BB659706DA45596" Ref="JX801"  Part="1"
-AR Path="/5C109CCF/6BB659706DA45596" Ref="JX801"  Part="1"
-F 0 "JX801" H 6200 1630 42  0000 L BNN
-F 1 "HEADER-3X1BOARDEDGE-SHORT" H 6200 1120 42  0000 L BNN
-F 2 "PX4FMUv2.4.6:HEADER_3X01_SMD_H_BOARD_EDGE_SHORT" H 6300 1300 50  0001 C CNN
-F 3 "" H 6300 1300 50  0001 C CNN
-	1    6300 1300
-	1    0    0    -1
-$EndComp
-$Comp
-L PX4FMUv2.4.6-eagle-import:GND #GND19
-U 1 0 906FD9F448B3EBD8
-P 5900 1500
-AR Path="/906FD9F448B3EBD8" Ref="#GND19"  Part="1"
-AR Path="/5C109CCF/906FD9F448B3EBD8" Ref="#GND019"  Part="1"
-F 0 "#GND019" H 5900 1500 50  0001 C CNN
-F 1 "GND" H 5800 1400 59  0000 L BNN
-F 2 "" H 5900 1500 50  0001 C CNN
-F 3 "" H 5900 1500 50  0001 C CNN
-	1    5900 1500
-	1    0    0    -1
-$EndComp
-$Comp
 L PX4FMUv2.4.6-eagle-import:DIODE-TVS D801
 U 1 0 B412B370257C0288
@@
 Text Notes 3200 2100 0    42   ~ 0
 Routed to FMU for debug purposes
-Text Notes 6200 800  0    59   ~ 0
-IO_SERIAL1
 Text Notes 6400 5000 0    59   ~ 0
 Spektrum/DSM
