File: PX4FMUv2.4.6_9.sch (KiCad schematic (older format))
At the start: 32 parts, among them J901 HEADER-3X163X16RA, U901 TXS0108QFN20, U902 TXS0108QFN20, U903 74LVC2G240

Commit message: removed some things
Parts:
- removed C901: 0u1, PX4FMUv2.4.6:0402-CAP, symbol PX4FMUv2.4.6-eagle-import:CAP0402
- removed D901, D902: PESD0402-140, PX4FMUv2.4.6:0402-TVS, symbol PX4FMUv2.4.6-eagle-import:DIODE-TVS
- removed unit 3 of J901
- removed unit 1 of J901
- removed unit 18 of J901
- removed R901: 10K, PX4FMUv2.4.6:0402-RES, symbol PX4FMUv2.4.6-eagle-import:RESISTOR0402-RES
- removed R909, R910: 220R, PX4FMUv2.4.6:0402-RES, symbol PX4FMUv2.4.6-eagle-import:RESISTOR0402-RES
- removed U903: 74LVC2G240, PX4FMUv2.4.6:TSSOP8_SOT505-2, symbol PX4FMUv2.4.6-eagle-import:74LVC2G240-TSSOP-8
Other:
- note removed: "S.Bus in/out"

Commit message: removed more things
Parts:
- removed C902: 0u1, PX4FMUv2.4.6:0402-CAP, symbol PX4FMUv2.4.6-eagle-import:CAP0402
- removed unit 14 of J901
- removed unit 15 of J901
- removed unit 12 of J901
- removed unit 13 of J901
- removed unit 16 of J901
- removed unit 17 of J901
- removed R902, R903, R904, R911, R912, R913: 220R, PX4FMUv2.4.6:0402-RES, symbol PX4FMUv2.4.6-eagle-import:RESISTOR0402-RES
- removed U901: TXS0108QFN20, PX4FMUv2.4.6:QFN20-RGY, symbol PX4FMUv2.4.6-eagle-import:TXS0108QFN20
Other:
- note removed: "Servo outputs"
